File: Kicad/RoboPower.kicad_pcb (KiCad board)
At the start: 2 copper layers, 101.6 x 53.3 mm, 58 parts, among them P1 Digital, P10 CONN_01X01, P11 CONN_01X01, P12 CONN_01X01, P13 CONN_01X01, P14 CONN_01X03, P15 CONN_01X03, P16 CONN_01X07, P17 CONN_01X03, P18 CONN_01X03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

Commit message: Work In Progress
Varius improvment
Parts:
- added P19: CONN_01X04, Pin_Headers:Pin_Header_Straight_1x04, F.Cu at (175.6, 49.4)
- R11, R9: value 150K -> 47K0
- R13, R15: value 47K -> 150K0
- R18, R20, R22, R24: footprint Resistors_ThroughHole:Resistor_Vertical_RM5mm -> Resistors_ThroughHole:Resistor_Horizontal_RM10mm
Connections:
- P14 pad 1: +5V -> GND
- P14 pad 3: GND -> +5V
- P15 pad 1: +5V -> GND
- P15 pad 3: GND -> +5V
- P16 pad 5: SDA -> SDA1
- P16 pad 6: SCL -> SCL1
- P17 pad 1: +5V -> GND
- P17 pad 3: GND -> +5V
- P18 pad 1: +5V -> GND
- P18 pad 3: GND -> +5V
- P5 pad 1: SCL -> SCL1
- P5 pad 2: SDA -> SDA1
- P7 pad 7: (no net) -> SDA
- P7 pad 8: (no net) -> SCL
Routing:
- net GND: track 103.2 -> 6.13 mm, vias 2 -> 0
- net SCL: track 34.9 -> 0.00 mm
- net SCL1: track 0.00 -> 34.2 mm
- net SDA: track 34.0 -> 0.00 mm
- net SDA1: track 0.00 -> 33.3 mm
- net +5V: track 5.54 -> 2.54 mm
- net ACP: track 28.8 -> 28.3 mm
